Commit message: odomを出力できるようにした(/ground_truth/odom)

File: src/scout_mini_description/install/scout_mini_description/share/scout_mini_description/urdf/scout_mini_gazebo.xacro (robot description, xacro)
@@ -28,4 +28,16 @@
       <mu2>1.0</mu2>
     </gazebo>
+    <gazebo reference="base_link">
+      <plugin name="ground_truth_p3d" filename="libgazebo_ros_p3d.so">
+        <ros>
+          <namespace>/</namespace>
+          <remapping>~/odom:=/ground_truth/odom</remapping>
+        </ros>
+        <update_rate>50.0</update_rate>
+        <frame_name>world</frame_name>
+        <body_name>base_link</body_name>
+        <gaussian_noise>0.0</gaussian_noise>
+      </plugin>
+    </gazebo>
   </xacro:macro>
 </robot>

File: src/scout_mini_description/urdf/scout_mini.urdf.xacro (robot description, xacro)
@@ -11,4 +11,16 @@
     <plugin name="gazebo_ros2_control" filename="libgazebo_ros2_control.so">
       <parameters>$(arg ros2_control_yaml)</parameters>
+    </plugin>
+  </gazebo>
+  <gazebo>
+    <plugin name="ground_truth_p3d" filename="libgazebo_ros_p3d.so">
+      <ros>
+        <namespace>/</namespace>
+        <remapping>odom:=/ground_truth/odom</remapping>
+      </ros>
+      <update_rate>50.0</update_rate>
+      <frame_name>world</frame_name>
+      <body_name>base_link</body_name>
+      <gaussian_noise>0.0</gaussian_noise>
     </plugin>
   </gazebo>

File: src/scout_mini_description/urdf/scout_mini_base.xacro (robot description, xacro)
@@ -18,4 +18,6 @@
           izz="3.431465"/>
       </inertial>
+    </link>
+    <link name="base_visual">
       <visual>
         <origin rpy="1.57 0 -1.57" xyz="0 0 0"/>
@@ -31,4 +33,9 @@
       </collision>
     </link>
+    <joint name="base_link_to_visual" type="fixed">
+      <parent link="base_link"/>
+      <child link="base_visual"/>
+      <origin xyz="0 0 0" rpy="0 0 0"/>
+    </joint>
     <link name="inertial_link">
       <inertial>
